File: Micromouse_V01 PCB/Micromouse_V01/Micromouse_V01.kicad_pcb (KiCad board)
At the start: 2 copper layers, 70.7 x 100 mm, 73 parts, among them J1 Conn_01x02_Female, J2 Conn_01x02_Female, J3 OLED, J4 Conn_01x02_Female, J5 AS5600 Left, J6 AS5600 Right, J7 Conn_01x02_Female, J8 Conn_01x02_Female, Q1 Q_NPN_BEC, Q2 Q_NPN_BEC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

Commit message: backup after long time, to update kicad
Other:
- net class Default removed
